Commit message: [jsk_fetch_startup] update head_l515 parameters

File: jsk_fetch_robot/jsk_fetch_startup/robots/head_l515.urdf.xacro (robot description, xacro)
@@ -10,5 +10,5 @@
       <origin rpy="0 0 0" xyz="0 0 0" />
       <geometry>
-        <mesh filename="package://jsk_fetch_accessories/head_l515/fetch_head_l515_mount_simplified.stl" scale="0.001 0.001 0.001" />
+        <mesh filename="package://jsk_fetch_accessories/head_l515/fetch_head_l515_mount.stl" scale="0.001 0.001 0.001" />
       </geometry>
       <material name="">
@@ -24,13 +24,13 @@
   </link>
   <joint name="head_l515_mount_virtual_joint" type="fixed">
-    <origin rpy="0 0 0" xyz="0 0 0" />
-    <parent link="head_pitch_link" />
+    <origin rpy="0 0 0" xyz="0.0255 0 0.055" />
+    <parent link="head_tilt_link" />
     <child link="head_l515_mount_link" />
   </joint>
-  <link name="head_l515_link"/>
+  <link name="head_l515_base_link"/>
   <joint name="head_l515_virtual_joint" type="fixed">
-    <origin rpy="0 0 0" xyz="0 0 0" />
+    <origin rpy="0 0 0" xyz="0.0095 0 0.01485" />
     <parent link="head_l515_mount_link" />
-    <child link="head_l515_link" />
+    <child link="head_l515_base_link" />
   </joint>
 </robot>

Commit message: [jsk_fetch_startup] fix l515 urdf parameter

File: jsk_fetch_robot/jsk_fetch_startup/robots/head_l515.urdf.xacro (robot description, xacro)
@@ -28,9 +28,9 @@
     <child link="head_l515_mount_link" />
   </joint>
-  <link name="head_l515_base_link"/>
+  <link name="l515_head_link"/>
   <joint name="head_l515_virtual_joint" type="fixed">
     <origin rpy="0 0 0" xyz="0.0095 0 0.01485" />
     <parent link="head_l515_mount_link" />
-    <child link="head_l515_base_link" />
+    <child link="l515_head_link" />
   </joint>
 </robot>
